File: SmartNeonPSU-Coilcraft/SmartNeonPSU.kicad_pcb (KiCad board)
At the start: 2 copper layers, 64 x 81.1 mm, 93 parts, among them J1 12VDC, J2 POWER, J3 SERIAL+GPIO, J4 TPS_IO, J5 EXT_SW, J6 LAMP1+, J7 LAMP1-, Q1 MMSS8050, Q2 MMSS8050, Q3 IRF7303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

Commit message: Add docs, sync schematics with reality
Parts:
- C20: value 4.7 uF -> 10 uF
- C21: value 10 pF -> 22 pF
- C22: value 6800 pF -> 18000 pF
- R16: value 162K -> 287K
Changed lines of the file:
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@@
     (descr "Resistor SMD 0805 (2012 Metric), square (rectangular) end terminal, IPC_7351 nominal, (Body size source: IPC-SM-782 page 72, https://www.pcb-3d.com/wordpress/wp-content/uploads/ipc-sm-782a_amendment_1_and_2.pdf), generated with kicad-footprint-generator")
     (tags "resistor")
-    (property "MPN1" "RC0805FR-07162KL")
+    (property "MPN1" "RC0805FR-07287KL")
     (property "Sheetfile" "SmartNeonPSU.kicad_sch")
     (property "Sheetname" "")
@@
       (effects (font (size 1 1) (thickness 0.2)))
     )
-    (fp_text value "162K" (at 0 1.65) (layer "F.Fab")
+    (fp_text value "287K" (at 0 1.65) (layer "F.Fab")
       (effects (font (size 1 1) (thickness 0.15)))
     )
@@
     (descr "Capacitor SMD 0805 (2012 Metric), square (rectangular) end terminal, IPC_7351 nominal, (Body size source: IPC-SM-782 page 76, https://www.pcb-3d.com/wordpress/wp-content/uploads/ipc-sm-782a_amendment_1_and_2.pdf, https://docs.google.com/spreadsheets/d/1BsfQQcO9C6DZCsRaXUlFlo91Tg2WpOkGARC1WS5S8t0/edit?usp=sharing), generated with kicad-footprint-generator")
     (tags "capacitor")
-    (property "MPN1" "C2012X7R1H475K125AE")
+    (property "MPN1" "C2012X5R1V106K085AC")
     (property "Sheetfile" "SmartNeonPSU.kicad_sch")
     (property "Sheetname" "")
@@
       (effects (font (size 1 1) (thickness 0.2)))
     )
-    (fp_text value "4.7 uF" (at 0 1.68) (layer "F.Fab")
+    (fp_text value "10 uF" (at 0 1.68) (layer "F.Fab")
       (effects (font (size 1 1) (thickness 0.15)))
     )
@@
     (descr "Capacitor SMD 0805 (2012 Metric), square (rectangular) end terminal, IPC_7351 nominal, (Body size source: IPC-SM-782 page 76, https://www.pcb-3d.com/wordpress/wp-content/uploads/ipc-sm-782a_amendment_1_and_2.pdf, https://docs.google.com/spreadsheets/d/1BsfQQcO9C6DZCsRaXUlFlo91Tg2WpOkGARC1WS5S8t0/edit?usp=sharing), generated with kicad-footprint-generator")
     (tags "capacitor")
-    (property "MPN1" "CC0805KRX7R9BB682")
+    (property "MPN1" "CC0805KRX7R9BB183")
     (property "Sheetfile" "SmartNeonPSU.kicad_sch")
     (property "Sheetname" "")
@@
       (effects (font (size 1 1) (thickness 0.2)))
     )
-    (fp_text value "6800 pF" (at 0 1.68 90) (layer "F.Fab")
+    (fp_text value "18000 pF" (at 0 1.68 90) (layer "F.Fab")
       (effects (font (size 1 1) (thickness 0.15)))
     )
@@
     (descr "Capacitor SMD 1812 (4532 Metric), square (rectangular) end terminal, IPC_7351 nominal, (Body size source: IPC-SM-782 page 76, https://www.pcb-3d.com/wordpress/wp-content/uploads/ipc-sm-782a_amendment_1_and_2.pdf), generated with kicad-footprint-generator")
     (tags "capacitor")
-    (property "MPN1" "C4520C0G3F100F")
+    (property "MPN1" "C4520C0G3F220K")
     (property "Sheetfile" "SmartNeonPSU.kicad_sch")
     (property "Sheetname" "")
@@
       (effects (font (size 1 1) (thickness 0.2)) (justify mirror))
     )
-    (fp_text value "10 pF" (at 0 -2.2 90) (layer "B.Fab")
+    (fp_text value "22 pF" (at 0 -2.2 90) (layer "B.Fab")
       (effects (font (size 1 1) (thickness 0.15)) (justify mirror))
     )
