File: SmartNeonPSU-Coilcraft/SmartNeonPSU.kicad_sch (KiCad schematic)
At the start: 87 parts, among them J1 12VDC, J2 POWER, J3 SERIAL+GPIO, J4 TPS_IO, J5 EXT_SW, J6 LAMP1+, J7 LAMP1-, Q1 MMSS8050, Q2 MMSS8050, Q3 IRF7303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

Commit message: Add docs, sync schematics with reality
Parts:
- C20: value 4.7 uF -> 10 uF; MPN1 C2012X7R1H475K125AE -> C2012X5R1V106K085AC
- C21: value 10 pF -> 22 pF; MPN1 C4520C0G3F100F -> C4520C0G3F220K
- C22: value 6800 pF -> 18000 pF; MPN1 CC0805KRX7R9BB682 -> CC0805KRX7R9BB183
- R16: value 162K -> 287K; MPN1 RC0805FR-07162KL -> RC0805FR-07287KL
Changed lines of the file:
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@@
       (effects (font (size 1.27 1.27)) (justify left))
     )
-    (property "Value" "10 pF" (id 1) (at 253.365 133.35 0)
+    (property "Value" "22 pF" (id 1) (at 253.365 133.35 0)
       (effects (font (size 1.27 1.27)) (justify left))
     )
@@
       (effects (font (size 1.27 1.27)) hide)
     )
-    (property "MPN1" "C4520C0G3F100F" (id 4) (at 250.825 132.08 0)
+    (property "MPN1" "C4520C0G3F220K" (id 4) (at 250.825 132.08 0)
       (effects (font (size 1.27 1.27)) hide)
     )
@@
       (effects (font (size 1.27 1.27)) (justify left))
     )
-    (property "Value" "6800 pF" (id 1) (at 251.46 139.065 0)
+    (property "Value" "18000 pF" (id 1) (at 251.46 139.065 0)
       (effects (font (size 1.27 1.27)) (justify left))
     )
@@
       (effects (font (size 1.27 1.27)) hide)
     )
-    (property "MPN1" "CC0805KRX7R9BB682" (id 4) (at 250.825 141.605 0)
+    (property "MPN1" "CC0805KRX7R9BB183" (id 4) (at 250.825 141.605 0)
       (effects (font (size 1.27 1.27)) hide)
     )
@@
       (effects (font (size 1.27 1.27)) (justify left))
     )
-    (property "Value" "162K" (id 1) (at 158.115 119.38 0)
+    (property "Value" "287K" (id 1) (at 158.115 119.38 0)
       (effects (font (size 1.27 1.27)) (justify left))
     )
@@
       (effects (font (size 1.27 1.27)) hide)
     )
-    (property "MPN1" "RC0805FR-07162KL" (id 4) (at 156.845 113.03 0)
+    (property "MPN1" "RC0805FR-07287KL" (id 4) (at 156.845 113.03 0)
       (effects (font (size 1.27 1.27)) hide)
     )
@@
     )
     (pin "1")
-  )
-  (symbol (lib_id "Device:C") (at 224.155 131.445 0) (unit 1)
-    (in_bom yes) (on_board yes)
-    (property "Reference" "C20" (id 0) (at 226.695 130.175 0)
-      (effects (font (size 1.27 1.27)) (justify left))
-    )
-    (property "Value" "4.7 uF" (id 1) (at 226.695 132.715 0)
-      (effects (font (size 1.27 1.27)) (justify left))
-    )
-    (property "Footprint" "Capacitor_SMD:C_0805_2012Metric" (id 2) (at 225.1202 135.255 0)
-      (effects (font (size 1.27 1.27)) hide)
-    )
-    (property "Datasheet" "~" (id 3) (at 224.155 131.445 0)
-      (effects (font (size 1.27 1.27)) hide)
-    )
-    (property "MPN1" "C2012X7R1H475K125AE" (id 4) (at 224.155 131.445 0)
-      (effects (font (size 1.27 1.27)) hide)
-    )
-    (pin "1")
-    (pin "2")
   )
   (symbol (lib_id "Device:R") (at 71.628 139.7144 180) (unit 1)
@@
     )
     (property "MPN1" "MBR230S1F-7" (id 5) (at 52.07 27.94 0)
+      (effects (font (size 1.27 1.27)) hide)
+    )
+    (pin "1")
+    (pin "2")
+  )
+  (symbol (lib_id "Device:C") (at 224.155 131.445 0) (unit 1)
+    (in_bom yes) (on_board yes)
+    (property "Reference" "C20" (id 0) (at 226.695 130.175 0)
+      (effects (font (size 1.27 1.27)) (justify left))
+    )
+    (property "Value" "10 uF" (id 1) (at 226.695 132.715 0)
+      (effects (font (size 1.27 1.27)) (justify left))
+    )
+    (property "Footprint" "Capacitor_SMD:C_0805_2012Metric" (id 2) (at 225.1202 135.255 0)
+      (effects (font (size 1.27 1.27)) hide)
+    )
+    (property "Datasheet" "~" (id 3) (at 224.155 131.445 0)
+      (effects (font (size 1.27 1.27)) hide)
+    )
+    (property "MPN1" "C2012X5R1V106K085AC" (id 4) (at 224.155 131.445 0)
       (effects (font (size 1.27 1.27)) hide)
     )
@@
       (reference "C19") (unit 1) (value "47 uF") (footprint "Capacitor_SMD:C_0805_2012Metric")
     )
-    (path "/aa213ca8-3e06-4412-af52-3386c4fab9f9"
-      (reference "C20") (unit 1) (value "4.7 uF") (footprint "Capacitor_SMD:C_0805_2012Metric")
+    (path "/bcb59008-2dd3-4fe9-9ccc-8a2f90f23081"
+      (reference "C20") (unit 1) (value "10 uF") (footprint "Capacitor_SMD:C_0805_2012Metric")
     )
     (path "/449e3155-16ea-42e5-8b6a-0c318fc89476"
-      (reference "C21") (unit 1) (value "10 pF") (footprint "Capacitor_SMD:C_1808_4520Metric_Slot")
+      (reference "C21") (unit 1) (value "22 pF") (footprint "Capacitor_SMD:C_1808_4520Metric_Slot")
     )
     (path "/51b8c561-e459-4fac-a380-3761f1257871"
-      (reference "C22") (unit 1) (value "6800 pF") (footprint "Capacitor_SMD:C_0805_2012Metric")
+      (reference "C22") (unit 1) (value "18000 pF") (footprint "Capacitor_SMD:C_0805_2012Metric")
     )
     (path "/bc1c377b-a155-474a-a038-dbd44a4e7dd6"
@@
     )
     (path "/9a45920d-217a-4a92-b6c2-ecc141d16559"
-      (reference "R16") (unit 1) (value "162K") (footprint "Resistor_SMD:R_0805_2012Metric")
+      (reference "R16") (unit 1) (value "287K") (footprint "Resistor_SMD:R_0805_2012Metric")
     )
     (path "/097b057b-6f92-4820-a5b5-7281e3dc927b"
