File: SmartNeonPSU-Coilcraft-Notch/SmartNeonPSU.kicad_pcb (KiCad board)
At the start: 2 copper layers, 64 x 81.1 mm, 93 parts, among them J1 12VDC, J2 POWER, J3 SERIAL+GPIO, J4 TPS_IO, J5 EXT_SW, J6 LAMP1+, J7 LAMP1-, Q1 MMSS8050, Q2 MMSS8050, Q3 IRF7303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

Commit message: v2
Parts:
- removed H5: MountingHole_Pad, MountingHole:MountingHole_3.2mm_M3_Pad_Via
- removed the J1 at (130.9, 67.6)
- removed the REF** at (121.7, 65.2)
- removed SW3: CONTROL, SmartNeonPSU:E-Switch_R1966A‎_7mm_RA
- moved J4 21.9 mm to (179.0, 69.5), turned to 180 degrees
- moved QR***** 20.2 mm to (166.8, 66.0)
- moved J1 16.8 mm to (121.0, 67.0), turned to 180 degrees
- moved C1 14.8 mm to (135.2, 69.0), turned to 180 degrees
- moved REF** 12.6 mm to (131.2, 66.0)
- moved F1 10.2 mm to (132.8, 61.0), turned to 180 degrees
- moved D1 6.52 mm to (139.5, 61.7)
- renumbered J2 to J1, J3 to J2, J4 to J3, J5 to J4, J6 to J5, J7 to J6
Routing:
- net /GPIO2: track 139.5 -> 117.8 mm
- net /GPIO0: track 148.6 -> 128.5 mm
- net Net-(F1-Pad2): track 18.5 -> 10.2 mm
- net +12V: track 88.7 -> 84.7 mm, vias 19 -> 16
- net GND: vias 52 -> 54
Other:
- board size 64 x 81.1 mm -> 64 x 80.4 mm

Commit message: Add docs, sync schematics with reality
Parts:
- C20: value 4.7 uF -> 10 uF
- C21: value 10 pF -> 22 pF
- C22: value 6800 pF -> 18000 pF
- R16: value 162K -> 287K
Changed lines of the file:
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@@
     (descr "Resistor SMD 0805 (2012 Metric), square (rectangular) end terminal, IPC_7351 nominal, (Body size source: IPC-SM-782 page 72, https://www.pcb-3d.com/wordpress/wp-content/uploads/ipc-sm-782a_amendment_1_and_2.pdf), generated with kicad-footprint-generator")
     (tags "resistor")
-    (property "MPN1" "RC0805FR-07162KL")
+    (property "MPN1" "RC0805FR-07287KL")
     (property "Sheetfile" "SmartNeonPSU.kicad_sch")
     (property "Sheetname" "")
@@
       (effects (font (size 1 1) (thickness 0.2)))
     )
-    (fp_text value "162K" (at 0 1.65) (layer "F.Fab")
+    (fp_text value "287K" (at 0 1.65) (layer "F.Fab")
       (effects (font (size 1 1) (thickness 0.15)))
     )
@@
     (descr "Capacitor SMD 0805 (2012 Metric), square (rectangular) end terminal, IPC_7351 nominal, (Body size source: IPC-SM-782 page 76, https://www.pcb-3d.com/wordpress/wp-content/uploads/ipc-sm-782a_amendment_1_and_2.pdf, https://docs.google.com/spreadsheets/d/1BsfQQcO9C6DZCsRaXUlFlo91Tg2WpOkGARC1WS5S8t0/edit?usp=sharing), generated with kicad-footprint-generator")
     (tags "capacitor")
-    (property "MPN1" "C2012X7R1H475K125AE")
+    (property "MPN1" "C2012X5R1V106K085AC")
     (property "Sheetfile" "SmartNeonPSU.kicad_sch")
     (property "Sheetname" "")
@@
       (effects (font (size 1 1) (thickness 0.2)))
     )
-    (fp_text value "4.7 uF" (at 0 1.68) (layer "F.Fab")
+    (fp_text value "10 uF" (at 0 1.68) (layer "F.Fab")
       (effects (font (size 1 1) (thickness 0.15)))
     )
@@
     (descr "Capacitor SMD 0805 (2012 Metric), square (rectangular) end terminal, IPC_7351 nominal, (Body size source: IPC-SM-782 page 76, https://www.pcb-3d.com/wordpress/wp-content/uploads/ipc-sm-782a_amendment_1_and_2.pdf, https://docs.google.com/spreadsheets/d/1BsfQQcO9C6DZCsRaXUlFlo91Tg2WpOkGARC1WS5S8t0/edit?usp=sharing), generated with kicad-footprint-generator")
     (tags "capacitor")
-    (property "MPN1" "CC0805KRX7R9BB682")
+    (property "MPN1" "CC0805KRX7R9BB183")
     (property "Sheetfile" "SmartNeonPSU.kicad_sch")
     (property "Sheetname" "")
@@
       (effects (font (size 1 1) (thickness 0.2)))
     )
-    (fp_text value "6800 pF" (at 0 1.68 90) (layer "F.Fab")
+    (fp_text value "18000 pF" (at 0 1.68 90) (layer "F.Fab")
       (effects (font (size 1 1) (thickness 0.15)))
     )
@@
     (descr "Capacitor SMD 1812 (4532 Metric), square (rectangular) end terminal, IPC_7351 nominal, (Body size source: IPC-SM-782 page 76, https://www.pcb-3d.com/wordpress/wp-content/uploads/ipc-sm-782a_amendment_1_and_2.pdf), generated with kicad-footprint-generator")
     (tags "capacitor")
-    (property "MPN1" "C4520C0G3F100F")
+    (property "MPN1" "C4520C0G3F220K")
     (property "Sheetfile" "SmartNeonPSU.kicad_sch")
     (property "Sheetname" "")
@@
       (effects (font (size 1 1) (thickness 0.2)) (justify mirror))
     )
-    (fp_text value "10 pF" (at 0 -2.2 90) (layer "B.Fab")
+    (fp_text value "22 pF" (at 0 -2.2 90) (layer "B.Fab")
       (effects (font (size 1 1) (thickness 0.15)) (justify mirror))
     )
@@
   (gr_line (start 142 56.2) (end 142 72) (layer "Edge.Cuts") (width 0.1))
   (gr_arc (start 120 134.95) (mid 118.585786 134.364213) (end 118 132.949998) (layer "Edge.Cuts") (width 0.1))
-  (gr_arc (start 158 56.2) (mid 158.563655 54.92777) (end 159.906129 54.561659) (layer "Edge.Cuts") (width 0.1))
+  (gr_arc (start 158 56.2) (mid 158.563655 54.927771) (end 159.906129 54.561659) (layer "Edge.Cuts") (width 0.1))
   (gr_arc (start 174.999999 89.45) (mid 174.847138 90.214609) (end 174.41331 90.862518) (layer "Edge.Cuts") (width 0.1))
   (gr_line (start 120 134.95) (end 180 134.95) (layer "Edge.Cuts") (width 0.1))
