File: SmartNeonPSU-DIY/SmartNeonPSU.kicad_pcb (KiCad board)
At the start: 2 copper layers, 64 x 81.1 mm, 89 parts, among them J1 12VDC, J2 POWER, J3 SERIAL+GPIO, J4 TPS_IO, J5 EXT_SW, J6 LAMP1+, J7 LAMP1-, Q1 MMSS8050, Q2 MMSS8050, Q3 IRF7303, Q4 IRF7303, SW1 RESET, SW2 IO0, SW3 CONTROL, U1 AP2205-33Y, U2 TPS68000, U3 ESP32-WROOM-32D

Commit message: v2
Parts:
- added C5: 1 uF, Capacitor_SMD:C_0805_2012Metric, F.Cu at (174.7, 112.7)
- added JP1: ESP-ABR, Jumper:SolderJumper-2_P1.3mm_Bridged_RoundedPad1.0x1.5mm, B.Cu at (126.7, 121.5)
- added JP2: ESP-BC, Jumper:SolderJumper-2_P1.3mm_Bridged_RoundedPad1.0x1.5mm, B.Cu at (126.7, 116.4)
- added U1: TSOP382xx, OptoDevice:Vishay_MINICAST-3Pin, F.Cu at (178.2, 117.7)
- moved REF** 24.0 mm to (172.0, 63.7)
- moved J5 15.1 mm to (158.5, 61.7), turned to 160 degrees
- moved REF** 12.1 mm to (121.7, 65.2), turned to -70 degrees
- moved R13 7.81 mm to (127.0, 73.7), turned to 180 degrees
- moved Q1 7.80 mm to (175.2, 101.8)
- moved C17 7.80 mm to (175.2, 108.7)
- moved J3 7.80 mm to (179.0, 108.2)
- moved Q2 7.80 mm to (175.2, 94.2)
- moved R18 7.80 mm to (175.2, 98.0)
- moved R19 7.80 mm to (175.2, 105.7)
- moved TP2 4.47 mm to (132.5, 93.5)
- moved QR***** 2.95 mm to (133.5, 77.2)
- moved SW3 1.07 mm to (171.0, 62.0)
- moved TR1 0.71 mm to (157.0, 82.7)
- moved C22 0.25 mm to (134.5, 91.5)
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- renumbered C9 to C10, C10 to C11, C11 to C12, C12 to C13, C13 to C14, C14 to C15, C15 to C16, C16 to C17, C17 to C18, C18 to C19, C19 to C20, C20 to C21, C21 to C22, C5 to C6, C6 to C7, C7 to C8, C8 to C9, U1 to U2, U2 to U3, U3 to U4
Connections:
- U4 pad 10: /BC -> /ESP_ABR
- U4 pad 11: /TPS_EN -> /ESP_BC
- U4 pad 12: /GPIO27 -> /TPS_EN
Routing:
- net /GPI35: track 0.00 -> 41.7 mm, vias 0 -> 1
- net /BC: track 67.3 -> 44.7 mm, vias 2 -> 1
- net /ESP_ABR: track 0.00 -> 21.2 mm, vias 0 -> 1
- net /ESP_BC: track 0.00 -> 20.8 mm, vias 0 -> 1
- net +3V3: track 72.7 -> 84.0 mm
- net /GPIO5: track 85.9 -> 96.6 mm
- net /SC: track 25.3 -> 15.1 mm
- net /GPIO0: track 139.4 -> 148.6 mm
- net /ESP_EN: track 60.6 -> 69.1 mm
- net /GPIO1: track 68.2 -> 74.4 mm
- net /GPIO3: track 68.1 -> 73.4 mm
- net /ABR: track 46.7 -> 51.8 mm
- net /PH: track 19.3 -> 15.2 mm
- net /GPIO4: track 82.8 -> 78.9 mm, vias 2 -> 1
- net /VSEN: track 34.8 -> 33.6 mm
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Other:
- outline, holes or cut-outs redrawn
- board text added: "By @kbx81 - v2 - April 2022"
- board text added: "EN pull resistors: install only one of R2, R4, R5; do NOT install R4 with ESP32! Voltage dividers: R6 & R7 may replace RV1 and C3. R8 & R9 may replace RV2 and C6. Install only one of R1 and R3; use R3 only with ESP32! Do not install R6, R7 and RV1 for ESP32 DAC control of ABR. For ESP32-controlled dimming, do NOT install R9 & RV2; install only R8 to pull BBR high and short C7. Do not place R13 ex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"
- board text added: "GPIO0: Switch A GPIO2: Switch B GPIO5: Status LED GPIO25: TPS68000 ABR (DAC) GPIO26: TPS68000 BC (PWM) GPIO27: TPS68000 EN GPIO34: TPS68000 ~{FAULT} GPIO35: IR Receiver"
- board text removed: "By @kbx81 - v1 - March 2022"
- board text removed: "Install only one of R1 and R3; use R3 only with ESP32! EN pull resistors: install only one of R2, R4, R5; do NOT install R4 with ESP32! Voltage dividers: R6 & R7 may replace RV1 and C3. R8 & R9 may replace RV2 and C5. For ESP32-controlled dimming, do NOT install R9 & RV2; install only R8 to pull BBR high and short C6. Do not place R13 except for {dblquote}slave{dblquote} configurations (see RM)."

Commit message: Add docs, sync schematics with reality
Parts:
- C20: value 4.7 uF -> 10 uF
- C21: value 10 pF -> 22 pF
- C22: value 6800 pF -> 18000 pF
- R16: value 162K -> 287K
Changed lines of the file:
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@@
     (descr "Resistor SMD 0805 (2012 Metric), square (rectangular) end terminal, IPC_7351 nominal, (Body size source: IPC-SM-782 page 72, https://www.pcb-3d.com/wordpress/wp-content/uploads/ipc-sm-782a_amendment_1_and_2.pdf), generated with kicad-footprint-generator")
     (tags "resistor")
-    (property "MPN1" "RC0805FR-07162KL")
+    (property "MPN1" "RC0805FR-07287KL")
     (property "Sheetfile" "SmartNeonPSU.kicad_sch")
     (property "Sheetname" "")
@@
       (effects (font (size 1 1) (thickness 0.2)))
     )
-    (fp_text value "162K" (at 0 1.65) (layer "F.Fab")
+    (fp_text value "287K" (at 0 1.65) (layer "F.Fab")
       (effects (font (size 1 1) (thickness 0.15)))
     )
@@
     (descr "Capacitor SMD 0805 (2012 Metric), square (rectangular) end terminal, IPC_7351 nominal, (Body size source: IPC-SM-782 page 76, https://www.pcb-3d.com/wordpress/wp-content/uploads/ipc-sm-782a_amendment_1_and_2.pdf, https://docs.google.com/spreadsheets/d/1BsfQQcO9C6DZCsRaXUlFlo91Tg2WpOkGARC1WS5S8t0/edit?usp=sharing), generated with kicad-footprint-generator")
     (tags "capacitor")
-    (property "MPN1" "C2012X7R1H475K125AE")
+    (property "MPN1" "C2012X5R1V106K085AC")
     (property "Sheetfile" "SmartNeonPSU.kicad_sch")
     (property "Sheetname" "")
@@
       (effects (font (size 1 1) (thickness 0.2)))
     )
-    (fp_text value "4.7 uF" (at 0 1.68) (layer "F.Fab")
+    (fp_text value "10 uF" (at 0 1.68) (layer "F.Fab")
       (effects (font (size 1 1) (thickness 0.15)))
     )
@@
     (descr "Capacitor SMD 0805 (2012 Metric), square (rectangular) end terminal, IPC_7351 nominal, (Body size source: IPC-SM-782 page 76, https://www.pcb-3d.com/wordpress/wp-content/uploads/ipc-sm-782a_amendment_1_and_2.pdf, https://docs.google.com/spreadsheets/d/1BsfQQcO9C6DZCsRaXUlFlo91Tg2WpOkGARC1WS5S8t0/edit?usp=sharing), generated with kicad-footprint-generator")
     (tags "capacitor")
-    (property "MPN1" "CC0805KRX7R9BB682")
+    (property "MPN1" "CC0805KRX7R9BB183")
     (property "Sheetfile" "SmartNeonPSU.kicad_sch")
     (property "Sheetname" "")
@@
       (effects (font (size 1 1) (thickness 0.2)))
     )
-    (fp_text value "6800 pF" (at 0 1.68 90) (layer "F.Fab")
+    (fp_text value "18000 pF" (at 0 1.68 90) (layer "F.Fab")
       (effects (font (size 1 1) (thickness 0.15)))
     )
@@
     (descr "Capacitor SMD 1812 (4532 Metric), square (rectangular) end terminal, IPC_7351 nominal, (Body size source: IPC-SM-782 page 76, https://www.pcb-3d.com/wordpress/wp-content/uploads/ipc-sm-782a_amendment_1_and_2.pdf), generated with kicad-footprint-generator")
     (tags "capacitor")
-    (property "MPN1" "C4520C0G3F100F")
+    (property "MPN1" "C4520C0G3F220K")
     (property "Sheetfile" "SmartNeonPSU.kicad_sch")
     (property "Sheetname" "")
@@
       (effects (font (size 1 1) (thickness 0.2)) (justify mirror))
     )
-    (fp_text value "10 pF" (at 0 -2.2 90) (layer "B.Fab")
+    (fp_text value "22 pF" (at 0 -2.2 90) (layer "B.Fab")
       (effects (font (size 1 1) (thickness 0.15)) (justify mirror))
     )
